File: gps/ESP32-BOARD-GPS.0.sch (KiCad schematic (older format))
At the start: 84 parts, among them J1 PIR SENSOR, J10 CON_USB_GCT_USB4105_REVA, J12 Conn_01x09, J2 OLED-128X64, J6 BATT, J7 PROG, J8 UART, J9 SWITCH, Q1 MBT3904DW1, Q2 MIC94052YC6-TR, SW1 RST, SW2 EN, SW3 ON/OFF, U1 IC-BATT-CHARGER-MCP73834, U2 ESP32-WROOM-32U, U3 ADXL343, U4 ISL9110IRTNZ, U5 MIC280-3YM6-TR, U6 CH340C

Commit message: Update the design
Parts:
- removed B1, B2: BUT, Button_Switch_SMD:SW_Push_1P1T_NO_CK_KMR2, symbol Switch:SW_Push
- removed D5, D7: RED, LED_SMD:LED_0805_2012Metric, symbol Device:LED
- removed D6: IN-PI554FCH, 1KiCadLib:LED-DIGITAL-IN-PI554FCH, symbol 1KiCadLib:LED-DIGITAL-IN-PI554FCH
- removed J1: PIR SENSOR, Connector_PinSocket_2.54mm:PinSocket_1x03_P2.54mm_Vertical, symbol Connector_Generic:Conn_01x03
- removed J12: Conn_01x09, Connector_PinHeader_2.54mm:PinHeader_1x09_P2.54mm_Vertical, symbol Connector_Generic:Conn_01x09
- removed J2: OLED-128X64, Connector_PinSocket_2.54mm:PinSocket_1x04_P2.54mm_Vertical, symbol 1KiCadLib:OLED-128X64
- removed J8: UART, Connector_PinHeader_2.54mm:PinHeader_1x04_P2.54mm_Vertical, symbol Connector_Generic:Conn_01x04
- removed J9: SWITCH, Button_Switch_SMD:SW_DIP_SPSTx04_Slide_Copal_CHS-04A_W5.08mm_P1.27mm_JPin, symbol Connector_Generic:Conn_02x04_Counter_Clockwise
- removed R14, R15, R16, R17, R24, R25, R26: 10K, Resistor_SMD:R_0805_2012Metric, symbol Device:R_Small
- removed U2: ESP32-WROOM-32U, 1KiCadLib:ESP32-WROOM-32U, symbol 1KiCadLib:ESP32-WROOM-32U
- removed U3: ADXL343, Package_LGA:LGA-14_3x5mm_P0.8mm_LayoutBorder1x6y, symbol Sensor_Motion:ADXL343
- removed U5: MIC280-3YM6-TR, Package_TO_SOT_SMD:SOT-23-6, symbol 1KiCadLib:IC-SENSOR-TEMP-MIC280-3YM6-TR
- added AE1, AE3: Antenna, Connector_PinHeader_2.54mm:PinHeader_1x01_P2.54mm_Vertical, symbol Device:Antenna
- added AE2, AE4: Antenna_Shield, Connector_Coaxial:U.FL_Hirose_U.FL-R-SMT-1_Vertical, symbol Device:Antenna_Shield
- added C17: 1uF, Capacitor_SMD:C_0805_2012Metric, symbol Device:C_Small
- added J1: Conn_01x10, Connector_PinHeader_2.54mm:PinHeader_1x10_P2.54mm_Vertical, symbol Connector_Generic:Conn_01x10
- added J2: Conn_01x04, Connector_PinHeader_2.54mm:PinHeader_1x04_P2.54mm_Vertical, symbol Connector_Generic:Conn_01x04
- added JP10, JP11, JP12, JP13, JP14, JP15, JP6, JP7, JP8, JP9: WIRE, Jumper:SolderJumper-2_P1.3mm_Open_RoundedPad1.0x1.5mm, symbol Device:Jumper_NC_Small
- added Q3: FMMT491QTA, Package_TO_SOT_SMD:SOT-23, symbol Device:Q_NPN_BEC
- added Q4: MIC94052YC6-TR, Package_TO_SOT_SMD:SOT-363_SC-70-6, symbol 1KiCadLib:P-MOSFET-MIC94052
- added U2: IC_GPS_L86-M33, 1KiCadLib:IC_GPS_L86-M33, symbol 1KiCadLib:IC_GPS_L86-M33
- added U3: RF_LORA_RFM95W-915S2, 1KiCadLib:RF_LORA_RFM95W-915S2, symbol 1KiCadLib:RF_LORA_RFM95W-915S2
- added U5: ESP32-C3-WROOM-02-H4, 1KiCadLib:ESP32-C3-WROOM-02-H4, symbol 1KiCadLib:ESP32-C3-WROOM-02-H4
- C10: value 10uF -> 1uF; footprint Capacitor_SMD:C_1206_3216Metric -> Capacitor_SMD:C_0805_2012Metric; DESCRIPTION Multilayer Ceramic Capacitors MLCC - SMD/SMT 10uF+/-10% 25V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 -> Multilayer Ceramic Capacitors MLCC - SMD/SMT 0805 16VDC 1uF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; MANUFACTURER KEMET -> Taiyo Yuden; MPN C1206C106K8PAC -> EMK212B7105KG-T; Mouser 80-C1206C106K8PAC -> 963-EMK212B7105KG-T
- C11, C5, C7: value 100nF -> 10uF; footprint Capacitor_SMD:C_0603_1608Metric -> Capacitor_SMD:C_1206_3216Metric; DESCRIPTION Multilayer Ceramic Capacitors MLCC - SMD/SMT 16V 0.1uF X7R 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 -> Multilayer Ceramic Capacitors MLCC - SMD/SMT 10uF+/-10% 25V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; MPN C0603C104J4RAC -> C1206C106K8PAC; Mouser 80-C0603C104J4RAC -> 80-C1206C106K8PAC
- C12: value 1uF -> 100nF; footprint Capacitor_SMD:C_0805_2012Metric -> Capacitor_SMD:C_0603_1608Metric; DESCRIPTION Multilayer Ceramic Capacitors MLCC - SMD/SMT 0805 16VDC 1uF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 -> Multilayer Ceramic Capacitors MLCC - SMD/SMT 16V 0.1uF X7R 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; MANUFACTURER Taiyo Yuden -> KEMET; MPN EMK212B7105KG-T -> C0603C104J4RAC; Mouser 963-EMK212B7105KG-T -> 80-C0603C104J4RAC
- C3: value 100nF -> 1uF; footprint Capacitor_SMD:C_0603_1608Metric -> Capacitor_SMD:C_0805_2012Metric; DESCRIPTION Multilayer Ceramic Capacitors MLCC - SMD/SMT 16V 0.1uF X7R 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 -> Multilayer Ceramic Capacitors MLCC - SMD/SMT 0805 16VDC 1uF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; MANUFACTURER KEMET -> Taiyo Yuden; MPN C0603C104J4RAC -> EMK212B7105KG-T; Mouser 80-C0603C104J4RAC -> 963-EMK212B7105KG-T
- R12, R18, R19, R20, R21, R22, R5, R6, R9: DESCRIPTION Thick Film Resistors - SMD ResHighPower 0805 10k 1% 1/2W TC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 -> Thick Film Resistors - SMD 10K 1%; MPN CHP0805-FX-1002ELF -> CR0805-FX-1002ELF; Mouser 652-CHP0805FX1002ELF -> 652-CR0805FX-1002ELF
- R13: value 10K -> 1.5K; DESCRIPTION Thick Film Resistors - SMD ResHighPower 0805 10k 1% 1/2W TC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 -> Thick Film Resistors - SMD 1/4W 1.5Kohms 1% 100ppm; MANUFACTURER Bourns -> Vishay / Dale; MPN CHP0805-FX-1002ELF -> RCC08051K50FKEA; Mouser 652-CHP0805FX1002ELF -> 71-RCC08051K50FKEA
- R4: value 1.5K -> 4.7K; DESCRIPTION Thick Film Resistors - SMD 1/4W 1.5Kohms 1% 100ppm -> Résistances à couches épaisses - CMS CRGCQ 0805 4K7 1% SMD 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; MANUFACTURER Vishay / Dale -> TE Connectivity / Holsworthy; MPN RCC08051K50FKEA -> CRGCQ0805F4K7; Mouser 71-RCC08051K50FKEA -> 279-CRGCQ0805F4K7
- R7: value 1.5K -> 47K; DESCRIPTION Thick Film Resistors - SMD 1/4W 1.5Kohms 1% 100ppm -> Résistances à couches épaisses - CMS CRGCQ 0805 47K 1% SMD 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; MANUFACTURER Vishay / Dale -> TE Connectivity / Holsworth; MPN RCC08051K50FKEA -> CRGCQ0805F47K; Mouser 71-RCC08051K50FKEA -> 279-CRGCQ0805F47K
- R8: value 1.5K -> 10K; DESCRIPTION Thick Film Resistors - SMD 1/4W 1.5Kohms 1% 100ppm -> Thick Film Resistors - SMD 10K 1%; MANUFACTURER Vishay / Dale -> Bourns; MPN RCC08051K50FKEA -> CR0805-FX-1002ELF; Mouser 71-RCC08051K50FKEA -> 652-CR0805FX-1002ELF
Connections:
- net labels added: GPS_FO, GPS_ON_OFF, GPS_RST, GPS_RX, GPS_TX, IO18, IO19, IO3, IO4_U2RXD, IO5_U2TXD, IO6, MCU_CS, MCU_MISO, MCU_MOSI, MCU_SCK, RF_MISO, RF_MOSI, RF_NSS, RF_RST, RF_SCK
- net labels removed: B1, B2, INT, IO12, IO13_ADC2_CH4_NTC, IO14, IO15_PIR_IN, IO16_U2RXD, IO17_U2TXD, IO2, IO21_I2C_SDA, IO22_I2C_SCL, IO4, LED2, LED3, LED4, LED_IN, S1, S2, S3, S4, SCL, SDA, VN, VP
- wire segments 368 -> 334
- no-connect marks 27 -> 18
Other:
- moved on the sheet: C1, C13, C14, C15, C16, C2, C6, C8, C9, D1, D2, D3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
