File: v2.0/ESP32-BOARD-V2.0.kicad_pcb (KiCad board)
At the start: 4 copper layers, 70 x 45 mm, 84 parts, among them J1 PIR SENSOR, J10 CON_USB_GCT_USB4105_REVA, J2 OLED-128X64, J3 PIR SENSOR, J4 PIR SENSOR, J5 PIR SENSOR, J6 BATT, J7 PROG, J8 UART, J9 SWITCH, Q1 MBT3904DW1, Q2 MIC94052YC6-TR, SW1 RST, SW2 EN, SW3 ON/OFF, U1 IC-BATT-CHARGER-MCP73834, U2 ESP32-WROOM-32U, U3 ADXL343, U4 ISL9110IRTNZ, U5 MIC280-3YM6-TR, U6 CH340C

Commit message: Update the design
Parts:
- removed the J3 at (158.1, 86.6)
- removed the J4 at (158.1, 78.4)
- added C4: 100nF, Capacitor_SMD:C_0603_1608Metric, F.Cu at (96.5, 69.5)
- added JP3: WIRE, Jumper:SolderJumper-2_P1.3mm_Open_RoundedPad1.0x1.5mm, B.Cu at (150.2, 95.8)
- J4: renamed from J6; footprint Connector_JST:JST_EH_B2B-EH-A_1x02_P2.50mm_Vertical -> Connector_JST:JST_XH_B2B-XH-A_1x02_P2.50mm_Vertical
- J5: value PIR SENSOR -> Conn_01x09; footprint Connector_PinSocket_2.54mm:PinSocket_1x03_P2.54mm_Vertical -> Connector_PinHeader_2.54mm:PinHeader_1x09_P2.54mm_Vertical
- moved J5 15.4 mm to (157.9, 79.3)
- moved J4 5.75 mm to (94.2, 96.0)
- moved C2 4.31 mm to (96.2, 71.5), turned to 180 degrees
- moved C1 3.25 mm to (92.2, 72.8), turned to 90 degrees
- moved J1 0.40 mm to (157.9, 70.5)
- renumbered C6 to C10, C7 to C11, C13 to C12, C14 to C13, C15 to C14, C8 to C15, C9 to C16, C4 to C5, C10 to C6, C11 to C7, C5 to C8, C12 to C9, D3 to D1, D1 to D2, D2 to D3, D7 to D6, D6 to D7, J7 to J3, J8 to J6, J9 to J7, J10 to J8, JP3 to JP4, JP4 to JP5, R3 to R1, R1 to R2, R21 to R20, R20 to R21, R2 to R3, R7 to R5, R5 to R6, R6 to R7
Connections:
- net Net-(J10-PadA6) renamed /D+
- net Net-(J10-PadA7) renamed /D-
- D6 pad 2: LED4 -> Net-(D6-Pad2)
- J5 pad 1: IO2 -> +3V3
- J5 pad 2: IO4 -> VP
- J5 pad 3: GND -> VN
- U2 pad 4: Net-(U2-Pad4) -> VP
- U2 pad 5: Net-(U2-Pad5) -> VN
Routing:
- net VBUS: track 59.0 -> 109.6 mm, vias 2 -> 4
- net VN: track 0.00 -> 43.2 mm, vias 0 -> 1
- net VP: track 0.00 -> 42.6 mm, vias 0 -> 1
- net +BATT: track 0.00 -> 36.0 mm, vias 4 -> 5
- net LED4: track 46.4 -> 74.0 mm, vias 2 -> 4
- net GND: track 73.2 -> 93.7 mm, vias 37 -> 47
- net Net-(R2-Pad1): track 0.00 -> 15.7 mm, vias 0 -> 2
- net Net-(D7-Pad2): track 0.00 -> 13.8 mm, vias 0 -> 1
- net Net-(R3-Pad1): track 0.00 -> 12.4 mm, vias 0 -> 2
- net /D+: track 9.11 -> 20.3 mm, vias 0 -> 2
- net Net-(JP5-Pad1): track 0.00 -> 9.07 mm, vias 0 -> 1
- net Net-(R6-Pad2): track 0.00 -> 9.03 mm
- net /D-: track 10.8 -> 19.4 mm, vias 0 -> 2
- net Net-(JP4-Pad1): track 0.00 -> 8.31 mm, vias 0 -> 1
- net IO14: track 50.2 -> 43.3 mm, vias 1 -> 2
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