File: v2.0/ESP32-BOARD-V2.0.sch (KiCad schematic (older format))
At the start: 84 parts, among them J1 PIR SENSOR, J10 CON_USB_GCT_USB4105_REVA, J2 OLED-128X64, J3 PIR SENSOR, J4 PIR SENSOR, J5 PIR SENSOR, J6 BATT, J7 PROG, J8 UART, J9 SWITCH, Q1 MBT3904DW1, Q2 MIC94052YC6-TR, SW1 RST, SW2 EN, SW3 ON/OFF, U1 IC-BATT-CHARGER-MCP73834, U2 ESP32-WROOM-32U, U3 ADXL343, U4 ISL9110IRTNZ, U5 MIC280-3YM6-TR, U6 CH340C

Commit message: Update the design
Parts:
- removed J3, J4, J5: PIR SENSOR, Connector_PinSocket_2.54mm:PinSocket_1x03_P2.54mm_Vertical, symbol Connector_Generic:Conn_01x03
- added C4: 100nF, Capacitor_SMD:C_0603_1608Metric, symbol Device:C_Small
- added J5: Conn_01x09, Connector_PinHeader_2.54mm:PinHeader_1x09_P2.54mm_Vertical, symbol Connector_Generic:Conn_01x09
- added JP3: WIRE, Jumper:SolderJumper-2_P1.3mm_Open_RoundedPad1.0x1.5mm, symbol Device:Jumper_NC_Small
- J4: renamed from J6; footprint Connector_JST:JST_EH_B2B-EH-A_1x02_P2.50mm_Vertical -> Connector_JST:JST_XH_B2B-XH-A_1x02_P2.50mm_Vertical
- renumbered C6 to C10, C7 to C11, C13 to C12, C14 to C13, C15 to C14, C8 to C15, C9 to C16, C4 to C5, C10 to C6, C11 to C7, C5 to C8, C12 to C9, D3 to D1, D1 to D2, D2 to D3, D7 to D6, D6 to D7, J7 to J3, J8 to J6, J9 to J7, J10 to J8, JP3 to JP4, JP4 to JP5, R3 to R1, R1 to R2, R21 to R20, R20 to R21, R2 to R3, R7 to R5, R5 to R6, R6 to R7
Connections:
- net labels added: D+, D-, VN, VP
- wire segments 367 -> 368
- no-connect marks 29 -> 27
Other:
- moved on the sheet: D1, D4, D5, D6, J4, R1, R4, R5, R8
